File: palcoder21.kicad_sch (KiCad schematic)
At the start: 27 parts, among them J1 Conn_01x10, J2 Conn_01x10, J3 Conn_01x01, J4 Conn_Coaxial, T1 2N2369, U1 82S129, U2 7474, U3 7404, U4 7407, Y1 8.86MHz

Commit message: Fix mistakes in first revision
Add missing trace

Fix swapped transistor pins

Use VCR instead of VNY
Parts:
- removed J3: Conn_01x01, Connector_PinHeader_2.54mm:PinHeader_1x01_P2.54mm_Horizontal, symbol Connector_Generic:Conn_01x01
- C2: value 22 -> 120pF
- R4: value 560 -> 120
Connections:
- net VNY is gone; now on net VCR: R4.2
- net VCC: now also T1.3 (C); no longer T1.1 (C)
- net VCR: now reaches J1.6 (Pin_6)
- net at L1.1, R9.1: now also T1.1 (E); no longer T1.3 (E)
- no-connect marks 12 -> 11
Changed lines of the file:
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@@
   (no_connect (at 81.28 140.97))
   (no_connect (at 81.28 153.67))
-  (no_connect (at 49.53 148.59))
   (no_connect (at 149.86 58.42))
   (no_connect (at 81.28 151.13))
@@
     (effects (font (size 1.27 1.27)) (justify left bottom))
   )
+  (label "VCR" (at 49.53 148.59 180)
+    (effects (font (size 1.27 1.27)) (justify right bottom))
+  )
   (label "VR" (at 93.98 96.52 180)
     (effects (font (size 1.27 1.27)) (justify right bottom))
@@
     (effects (font (size 1.27 1.27)) (justify right bottom))
   )
-  (label "VNY" (at 104.14 135.89 180)
-    (effects (font (size 1.27 1.27)) (justify right bottom))
-  )
   (label "VR" (at 49.53 140.97 180)
     (effects (font (size 1.27 1.27)) (justify right bottom))
@@
     (effects (font (size 1.27 1.27)) (justify left bottom))
   )
-  (label "VNY" (at 179.07 151.13 180)
+  (label "VCR" (at 179.07 151.13 180)
     (effects (font (size 1.27 1.27)) (justify right bottom))
   )
@@
     (in_bom yes) (on_board yes)
     (property "Reference" "R4" (id 0) (at 182.88 145.8722 90))
-    (property "Value" "560" (id 1) (at 182.88 148.1836 90))
+    (property "Value" "120" (id 1) (at 182.88 148.1836 90))
     (property "Footprint" "Resistor_THT:R_Axial_DIN0204_L3.6mm_D1.6mm_P7.62mm_Horizontal" (id 2) (at 182.88 149.352 90)
       (effects (font (size 1.27 1.27)) hide)
@@
     (pin "3")
   )
-  (symbol (lib_id "Connector_Generic:Conn_01x01") (at 109.22 135.89 0) (unit 1)
-    (in_bom yes) (on_board yes)
-    (property "Reference" "J3" (id 0) (at 111.252 134.8232 0)
-      (effects (font (size 1.27 1.27)) (justify left))
-    )
-    (property "Value" "Conn_01x01" (id 1) (at 111.252 137.1346 0)
-      (effects (font (size 1.27 1.27)) (justify left))
-    )
-    (property "Footprint" "Connector_PinHeader_2.54mm:PinHeader_1x01_P2.54mm_Horizontal" (id 2) (at 109.22 135.89 0)
-      (effects (font (size 1.27 1.27)) hide)
-    )
-    (property "Datasheet" "~" (id 3) (at 109.22 135.89 0)
-      (effects (font (size 1.27 1.27)) hide)
-    )
-    (pin "1")
-  )
   (symbol (lib_id "Device:C") (at 40.64 177.8 0) (unit 1)
     (in_bom yes) (on_board yes)
@@
       (effects (font (size 1.27 1.27)) (justify left))
     )
-    (property "Value" "22" (id 1) (at 198.501 145.923 0)
+    (property "Value" "120pF" (id 1) (at 198.501 145.923 0)
       (effects (font (size 1.27 1.27)) (justify left))
     )
@@
     )
     (path "/00000000-0000-0000-0000-0000613a08c8"
-      (reference "C2") (unit 1) (value "22") (footprint "Capacitor_THT:C_Disc_D5.1mm_W3.2mm_P5.00mm")
+      (reference "C2") (unit 1) (value "120pF") (footprint "Capacitor_THT:C_Disc_D5.1mm_W3.2mm_P5.00mm")
     )
     (path "/00000000-0000-0000-0000-000061388ae8"
@@
       (reference "J2") (unit 1) (value "Conn_01x10") (footprint "Connector_PinHeader_2.54mm:PinHeader_1x10_P2.54mm_Vertical")
     )
-    (path "/00000000-0000-0000-0000-000061386db4"
-      (reference "J3") (unit 1) (value "Conn_01x01") (footprint "Connector_PinHeader_2.54mm:PinHeader_1x01_P2.54mm_Horizontal")
-    )
     (path "/00000000-0000-0000-0000-0000613dae1f"
       (reference "J4") (unit 1) (value "Conn_Coaxial") (footprint "5413558-1:BNC_TEConnectivity_BNC_TEConnectivity_5413558-1")
@@
     )
     (path "/00000000-0000-0000-0000-000061327fe4"
-      (reference "R4") (unit 1) (value "560") (footprint "Resistor_THT:R_Axial_DIN0204_L3.6mm_D1.6mm_P7.62mm_Horizontal")
+      (reference "R4") (unit 1) (value "120") (footprint "Resistor_THT:R_Axial_DIN0204_L3.6mm_D1.6mm_P7.62mm_Horizontal")
     )
     (path "/00000000-0000-0000-0000-000061349cfd"
